File: pcb/poe-backplate/poe-backplate.kicad_pcb (KiCad board)
At the start: 6 copper layers, 59.2 x 75 mm, 113 parts, among them IC1 LAN9500A-ABZJ, IC2 93LC66AT-I_OT, J3 USB_C_Receptacle_USB2.0_14P, J4 USB_C_Receptacle_USB2.0_14P, J5 Conn_02x04_Counter_Clockwise, U1 LP38693MP-3.3, U2 HY931147C, U5 USBLC6-2SC6, Y1 ECS-250-18-36B2-CTY-TR

Commit message: small fixes of v0.3.1
Parts:
- removed kibuzzard-697F85DD: G***, kibuzzard-697F85DD
- removed kibuzzard-697F85E3: G***, kibuzzard-697F85E3
- added kibuzzard-69D3A526: G***, kibuzzard-69D3A526, F.Cu at (96.2, 109.0)
- added kibuzzard-69D3A52E: G***, kibuzzard-69D3A52E, F.Cu at (98.2, 109.0)
Routing:
- net /PoE/VDD33A: vias 7 -> 8
