File: pcb/poe-backplate/poe.kicad_sch (KiCad schematic)
At the start: 19 parts, among them U2 HY931147C

Commit message: PoE backplate
Parts:
- added D4: RCLAMP0524PATCT, RCLAMP0524PATCT, symbol RCLAMP0524PATCT:RCLAMP0524PATCT
Connections:
- net GND: now also D4.3 (GND_1), D4.8 (GND_2)
- net RXN: now also D4.4 (INPUT_LINES_3)
- net RXP: now also D4.5 (INPUT_LINES_4)
- net TXN: now also D4.1 (INPUT_LINES_1)
- net TXP: now also D4.2 (INPUT_LINES_2)
- net POE_VIN+: now reaches C24.1, POE1.1 (VIN+), U2.P$9 (V+)
- net POE_VIN-: now reaches C24.2, POE1.2 (VIN-), U2.P$10 (V-)
- no-connect marks 3 -> 7
Other:
- note added: "PoE Module"
- note added: "RJ45 + magnetics + TVS"
- note removed: "TODO: optional - Add TBS / ESD for eth data lines"
- moved on the sheet: C24, C25, D3, POE1, R15, R16, R17, R18, R19, TP10, TP11, TP7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
