File: pcb/poe-backplate/usb_to_ethernet.kicad_sch (KiCad schematic)
At the start: 65 parts, among them IC1 LAN9500A-ABZJ, IC2 93LC66AT-I_OT, J3 USB_C_Receptacle_USB2.0_14P, J4 USB_C_Receptacle_USB2.0_14P, J5 Conn_02x04_Counter_Clockwise, U1 LP38693MP-3.3, U5 USBLC6-2SC6, Y1 ECS-250-18-36B2-CTY-TR

Commit message: PoE backplate
Parts:
- added H1, H2, H3, H4: MountingHole_Pad, 9774030151R:9774030151R, symbol Mechanical:MountingHole_Pad
- added JP1: SolderJumper_3_Open, Jumper:SolderJumper-3_P1.3mm_Open_RoundedPad1.0x1.5mm_NumberLabels, symbol Jumper:SolderJumper_3_Open
- added S6: 218-2LPSTRF, 2182LPSTRF, symbol 218-2LPSTRF:218-2LPSTRF
- added SW1: power reset, Button_Switch_SMD:SW_SPST_PTS810, symbol Switch:SW_Push
- J5: value Conn_02x04_Counter_Clockwise -> Conn_02x12_Counter_Clockwise; footprint Connector_PinSocket_2.54mm:PinSocket_2x04_P2.54mm_Vertical -> Connector_PinHeader_2.54mm:PinHeader_2x12_P2.54mm_Vertical; symbol Connector_Generic:Conn_02x04_Odd_Even -> Connector_Generic:Conn_02x12_Odd_Even; DigiKey (none) -> 803-87-024-10-001101; FT Rotation Offset 90 -> (none); LCSC C2977588 -> (none); URL (none) -> https://www.digikey.es/en/products/detail/preci-dip/803-87-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; low profile (none) -> 415-83-212-41-001101
- R3, R5: LCSC C17168 -> C60490
Connections:
- net +3.3V: now also JP1.3 (B)
- net +5V: now also J5.16 (Pin_16), S6.3; no longer J5.7 (Pin_7)
- net GND: now also J5.15 (Pin_15), JP1.1 (A), S6.1, SW1.2; no longer J5.8 (Pin_8)
- net USBDN: now also J5.14 (Pin_14); no longer J5.5 (Pin_5), U5.6 (I/O1)
- net USBDP: now also J5.13 (Pin_13); no longer J5.6 (Pin_6), U5.4 (I/O2)
- net USB_OTG_SWITCH: now reaches J5.1 (Pin_1)
- net USB_OTG_SWITCH: now also JP1.2 (C)
- net GLOBAL_EN: now reaches J5.2 (Pin_2)
- net GLOBAL_EN: now also SW1.1
- net OTG_MODE_SW1: now reaches J5.3 (Pin_3)
- net OTG_MODE_SW1: now also S6.2
- net nRPIBOOT: now reaches J5.4 (Pin_4)
- net nRPIBOOT: now also S6.4
- new net EEPROM_nWP: J5.6 (Pin_6)
- new net SCL1: J5.10 (Pin_10)
- new net SDA1: J5.9 (Pin_9)
- new net SPI1_CS1: J5.24 (Pin_24)
- new net SPI1_CS2: J5.23 (Pin_23)
- new net SPI1_CS3: J5.21 (Pin_21)
- new net SPI1_MISO: J5.20 (Pin_20)
- new net SPI1_MOSI: J5.22 (Pin_22)
- new net SPI1_SCLK: J5.18 (Pin_18)
- new net UART_RX: J5.12 (Pin_12)
- new net UART_TX: J5.11 (Pin_11)
- new net USBD_POGO_N: J5.5 (Pin_5), U5.6 (I/O1)
- new net USBD_POGO_P: J5.7 (Pin_7), U5.4 (I/O2)
- no-connect marks 21 -> 25
Other:
- note added: "DIP switch"
- note added: "EEPROM mode OTG mode"
- note removed: "SCL"
- note removed: "SDA"
