File: pcb/wall-panel/RTC.kicad_sch (KiCad schematic)
At the start: 4 parts, among them J4 Conn_01x02_Socket, U5 DS3231M

Commit message: wall panel v0.3
Connections:
- net GND: now also J4.2 (Pin_2); no longer J4.1 (Pin_1)
- net at C17.1, U5.14 (VBAT): now also J4.1 (Pin_1); no longer J4.2 (Pin_2)
Other:
- company: Grigorii Merkushev (aka brushknight) -> dotstar.tech
- title: Wall panel -> Wall Panel
Changed lines of the file:
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@@
 	(paper "A3")
 	(title_block
-		(title "Wall panel")
-		(date "2026-01-09")
-		(rev "1")
-		(company "Grigorii Merkushev (aka brushknight)")
-		(comment 1 "brushknight.com")
+		(title "Wall Panel")
+		(date "2026-02-02")
+		(rev "v0.3")
+		(company "dotstar.tech")
+		(comment 1 "designed by Grigorii Merkushev (aka brushknight)")
+		(comment 2 "brushknight.com")
 	)
 	(text "RTC and RTC wakeup"
@@
 	(wire
 		(pts
+			(xy 66.04 45.72) (xy 66.04 49.53)
+		)
+		(stroke
+			(width 0)
+			(type default)
+		)
+	)
+	(wire
+		(pts
 			(xy 57.15 63.5) (xy 66.04 63.5)
-		)
-		(stroke
-			(width 0)
-			(type default)
-		)
-	)
-	(wire
-		(pts
-			(xy 66.04 49.53) (xy 66.04 45.72)
 		)
 		(stroke
@@
 		)
 		(instances
-			(project "CM4IOv5"
+			(project "wall_panel"
 				(path "/e63e39d7-6ac0-4ffd-8aa3-1841a4541b55/00000000-0000-0000-0000-00005e328d89"
 					(reference "#PWR070")
@@
 		)
 		(instances
-			(project "CM4IOv5"
+			(project "wall_panel"
 				(path "/e63e39d7-6ac0-4ffd-8aa3-1841a4541b55/00000000-0000-0000-0000-00005e328d89"
 					(reference "#PWR069")
@@
 		)
 		(instances
-			(project "CM4IOv5"
+			(project "wall_panel"
 				(path "/e63e39d7-6ac0-4ffd-8aa3-1841a4541b55/00000000-0000-0000-0000-00005e328d89"
 					(reference "C17")
@@
 		)
 		(instances
-			(project "CM4IOv5"
+			(project "wall_panel"
 				(path "/e63e39d7-6ac0-4ffd-8aa3-1841a4541b55/00000000-0000-0000-0000-00005e328d89"
 					(reference "#PWR025")
@@
 		)
 		(instances
-			(project "CM4IOv5"
+			(project "wall_panel"
 				(path "/e63e39d7-6ac0-4ffd-8aa3-1841a4541b55/00000000-0000-0000-0000-00005e328d89"
 					(reference "#PWR024")
@@
 	(symbol
 		(lib_id "Connector:Conn_01x02_Socket")
-		(at 71.12 49.53 0)
+		(at 71.12 52.07 0)
+		(mirror x)
 		(unit 1)
 		(exclude_from_sim no)
@@
 		(on_board yes)
 		(dnp no)
-		(fields_autoplaced yes)
 		(property "Reference" "J4"
-			(at 72.39 49.5299 0)
+			(at 72.39 52.0701 0)
 			(effects
 				(font
@@
 		)
 		(property "Value" "Conn_01x02_Socket"
-			(at 72.39 52.0699 0)
+			(at 72.39 49.5301 0)
 			(effects
 				(font
@@
 		)
 		(property "Footprint" "CONN02_533984002_MOL:CONN02_533984002_MOL"
-			(at 71.12 49.53 0)
+			(at 71.12 52.07 0)
 			(effects
 				(font
@@
 		)
 		(property "Datasheet" "https://www.molex.com/en-us/products/part-detail-pdf/533984002?display=pdf"
-			(at 71.12 49.53 0)
+			(at 71.12 52.07 0)
 			(effects
 				(font
@@
 		)
 		(property "Description" "Generic connector, single row, 01x02, script generated"
-			(at 71.12 49.53 0)
+			(at 71.12 52.07 0)
 			(effects
 				(font
@@
 		)
 		(property "URL" "https://eu.mouser.com/ProductDetail/Molex/53398-4002?qs=iLbezkQI%252BsjNR44XnvA9PQ%3D%3D&srsltid=AfmBOorTWWap8qiFVUOD5P7LnDBaNxt2k6tC8Z0wXPSvf5gvXqJPTJfT"
-			(at 71.12 49.53 0)
+			(at 71.12 52.07 0)
 			(effects
 				(font
@@
 		)
 		(property "LCSC" "C16076276"
-			(at 71.12 49.53 0)
+			(at 71.12 52.07 0)
 			(effects
 				(font
@@
 		)
 		(property "JLCPCB Rotation Offset" ""
-			(at 71.12 49.53 0)
-			(effects
-				(font
+			(at 71.12 52.07 0)
+			(effects
+				(font
