File: pcb/wall-panel/USB2-HUB.kicad_sch (KiCad schematic)
At the start: 38 parts, among them J1 USB_C_Receptacle_USB2.0_14P, J17 USB_C_Receptacle_USB2.0_14P, J2 USB_C_Receptacle_USB2.0_14P, U1 FSUSB42MUX, U2 USB2514B-I/M2, U3 TPD4EUSB30, U4 AP22653W6, Y1 ABM8G-24.000MHZ-18-D2Y-T

Commit message: wall panel v0.3
Other:
- company: Grigorii Merkushev (aka brushknight) -> dotstar.tech
- title: Wall panel -> Wall Panel
Changed lines of the file:
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@@
 	(paper "A3")
 	(title_block
-		(title "Wall panel")
-		(date "2026-01-09")
-		(rev "1")
-		(company "Grigorii Merkushev (aka brushknight)")
-		(comment 1 "brushknight.com")
+		(title "Wall Panel")
+		(date "2026-02-02")
+		(rev "v0.3")
+		(company "dotstar.tech")
+		(comment 1 "designed by Grigorii Merkushev (aka brushknight)")
+		(comment 2 "brushknight.com")
 	)
 	(text "J17,USB_C_Receptacle_GCT_USB4105-xx-A_16P_TopMnt_Horizontal,1,USB_C_Receptacle_USB2.0_14P,C136423"
@@
 		)
 		(instances
-			(project "CM4IOv5"
+			(project "wall_panel"
 				(path "/e63e39d7-6ac0-4ffd-8aa3-1841a4541b55/00000000-0000-0000-0000-00005e072e02"
 					(reference "R26")
@@
 		)
 		(instances
-			(project "CM4IOv5"
+			(project "wall_panel"
 				(path "/e63e39d7-6ac0-4ffd-8aa3-1841a4541b55/00000000-0000-0000-0000-00005e072e02"
 					(reference "#PWR014")
@@
 		)
 		(instances
-			(project "CM4IOv5"
+			(project "wall_panel"
 				(path "/e63e39d7-6ac0-4ffd-8aa3-1841a4541b55/00000000-0000-0000-0000-00005e072e02"
 					(reference "R9")
@@
 		)
 		(instances
-			(project "CM4IOv5"
+			(project "wall_panel"
 				(path "/e63e39d7-6ac0-4ffd-8aa3-1841a4541b55/00000000-0000-0000-0000-00005e072e02"
 					(reference "R25")
@@
 		)
 		(instances
-			(project "CM4IOv5"
+			(project "wall_panel"
 				(path "/e63e39d7-6ac0-4ffd-8aa3-1841a4541b55/00000000-0000-0000-0000-00005e072e02"
 					(reference "R8")
@@
 		)
 		(instances
-			(project "CM4IOv5"
+			(project "wall_panel"
 				(path "/e63e39d7-6ac0-4ffd-8aa3-1841a4541b55/00000000-0000-0000-0000-00005e072e02"
 					(reference "#PWR082")
@@
 		)
 		(instances
-			(project "CM4IOv5"
+			(project "wall_panel"
 				(path "/e63e39d7-6ac0-4ffd-8aa3-1841a4541b55/00000000-0000-0000-0000-00005e072e02"
 					(reference "J17")
@@
 		)
 		(instances
-			(project "CM4IOv5"
+			(project "wall_panel"
 				(path "/e63e39d7-6ac0-4ffd-8aa3-1841a4541b55/00000000-0000-0000-0000-00005e072e02"
 					(reference "#PWR083")
@@
 		)
 		(instances
-			(project "CM4IOv5"
+			(project "wall_panel"
 				(path "/e63e39d7-6ac0-4ffd-8aa3-1841a4541b55/00000000-0000-0000-0000-00005e072e02"
 					(reference "J1")
@@
 		)
 		(instances
-			(project "CM4IOv5"
+			(project "wall_panel"
 				(path "/e63e39d7-6ac0-4ffd-8aa3-1841a4541b55/00000000-0000-0000-0000-00005e072e02"
 					(reference "#PWR081")
@@
 		)
 		(instances
-			(project "CM4IOv5"
+			(project "wall_panel"
 				(path "/e63e39d7-6ac0-4ffd-8aa3-1841a4541b55/00000000-0000-0000-0000-00005e072e02"
 					(reference "#PWR03")
@@
 		)
 		(instances
-			(project "CM4IOv5"
+			(project "wall_panel"
 				(path "/e63e39d7-6ac0-4ffd-8aa3-1841a4541b55/00000000-0000-0000-0000-00005e072e02"
 					(reference "#PWR061")
@@
 		)
 		(instances
-			(project "CM4IOv5"
+			(project "wall_panel"
 				(path "/e63e39d7-6ac0-4ffd-8aa3-1841a4541b55/00000000-0000-0000-0000-00005e072e02"
 					(reference "R12")

Commit message: pogo pins wall panel
Parts:
- added C34: 100n, Capacitor_SMD:C_0402_1005Metric, symbol Device:C
- added IC1: TS3USB221RSER, TS3USB221RSER:RSE_R-PUQFN-N10_, symbol TS3USB221RSER:TS3USB221RSER
- added R17: 100K, Resistor_SMD:R_0402_1005Metric, symbol Device:R
- added U13: TPD4EUSB30, Package_SON:USON-10_2.5x1.0mm_P0.5mm, symbol CM4IO:TPD4EUSB30
- J1, J2: footprint Connector_USB:USB_C_Receptacle_G-Switch_GT-USB-7051x -> Connector_USB:USB_C_Receptacle_GCT_USB4105-xx-A_16P_TopMnt_Horizontal; LCSC C2843970 -> C136423
Connections:
- net +3.3V: now also C34.1, IC1.10 (VCC), R17.1
- net GND: now also C34.2, IC1.4 (~{OE}), IC1.5 (GND), U13.3 (GND), U13.8 (GND); no longer J1.S1 (SHIELD), J17.S1 (SHIELD), J2.S1 (SHIELD)
- net HD1_N: now also J17.A7 (D-), J17.B7 (D-); no longer J2.A7 (D-), J2.B7 (D-)
- net HD1_P: now also J17.A6 (D+), J17.B6 (D+); no longer J2.A6 (D+), J2.B6 (D+)
- net HD4_N: now also J2.A7 (D-), J2.B7 (D-); no longer J17.A7 (D-), J17.B7 (D-)
- net HD4_P: now also J2.A6 (D+), J2.B6 (D+); no longer J17.A6 (D+), J17.B6 (D+)
- net USBD_N: now also IC1.3 (D-); no longer J1.A7 (D-), J1.B7 (D-), U3.4 (D2+), U3.7
- net USBD_P: now also IC1.2 (D+); no longer J1.A6 (D+), J1.B6 (D+), U3.5 (D2-), U3.6
- net OTG_5V renamed VBUS_IN
- new net: U13.1 (D1+), U13.10
- new net: U13.2 (D1-), U13.9
- new net USBD_OTG_N: IC1.6 (2D-), J1.A7 (D-), J1.B7 (D-), U3.5 (D2-), U3.6
- new net USBD_OTG_P: IC1.7 (2D+), J1.A6 (D+), J1.B6 (D+), U3.4 (D2+), U3.7
- new net USBD_POGO_N: IC1.8 (1D-), U13.5 (D2-), U13.6
- new net USBD_POGO_P: IC1.9 (1D+), U13.4 (D2+), U13.7
- new net USB_OTG_SWITCH: IC1.1 (S), R17.2
