File: pcb/wall-panel/USB2-HUB.kicad_sch (KiCad schematic)
At the start: 42 parts, among them IC1 TS3USB221RSER, J1 USB_C_Receptacle_USB2.0_14P, J17 USB_C_Receptacle_USB2.0_14P, J2 USB_C_Receptacle_USB2.0_14P, U1 FSUSB42MUX, U13 TPD4EUSB30, U2 USB2514B-I/M2, U3 TPD4EUSB30, U4 AP22653W6, Y1 ABM8G-24.000MHZ-18-D2Y-T

Commit message: wall panel rev 5
Other:
- note added: "ESD protection"
- note added: "POGO pins USB ESD protection"
- note added: "Side USB Out"
- note added: "USB in ESD protection"
- note added: "USB out power limiter"
- note added: "USB switch 2.0 + OTG mode"
- note added: "USB swith POGO/USB in"
- note removed: "J17,USB_C_Receptacle_GCT_USB4105-xx-A_16P_TopMnt_Horizontal,1,USB_C_Receptacle_USB2.0_14P,C136423"
- note removed: "Micro USB ESD protection"
- moved on the sheet: C1, C10, C11, C12, C13, C14, C15, C16, C2, C3, C34, C4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
