File: pcb/wall-panel/power.kicad_sch (KiCad schematic)
At the start: 3 parts

Commit message: wall panel v0.3
Parts:
- added C32, C33: 22uF, Capacitor_SMD:C_0805_2012Metric, symbol Device:C_Small
- added D3: B5817W, Diode_SMD:D_SOD-123, symbol Device:D
- added JP5, JP6: SolderJumper_2_Bridged, Jumper:SolderJumper-2_P1.3mm_Bridged2Bar_Pad1.0x1.5mm, symbol Jumper:SolderJumper_2_Bridged
- added JP7, JP8: 12.8/15V, Jumper:SolderJumper-3_P1.3mm_Bridged12_Pad1.0x1.5mm, symbol Jumper:SolderJumper_3_Bridged12
- added L1: 10uH, Inductor_SMD:L_Taiyo-Yuden_NR-40xx, symbol Device:L_Small
- added R17: 200K, Resistor_SMD:R_0402_1005Metric, symbol Device:R_Small
- added R18, R29: 10K, Resistor_SMD:R_0402_1005Metric, symbol Device:R_Small
- added R30: 240K, Resistor_SMD:R_0402_1005Metric, symbol Device:R_Small
- added TP3: boost in, TestPoint:TestPoint_Pad_D1.5mm, symbol Connector:TestPoint
- added TP4: boost out, TestPoint:TestPoint_Pad_D1.5mm, symbol Connector:TestPoint
- added TP5: boost fb, TestPoint:TestPoint_Pad_D1.5mm, symbol Connector:TestPoint
- added U11: MT3608, Package_TO_SOT_SMD:SOT-23-6, symbol Regulator_Switching:MT3608
Connections:
- net +5V: now also JP5.1 (A)
- new net: C32.1, D3.1 (K), JP6.1 (A), JP7.2 (C)
- new net: JP8.1 (A), R29.1
- new net: R17.1, R18.2, R29.2, R30.1, TP5.1, U11.3 (FB)
- new net: JP8.3 (B), R18.1
- new net: JP7.1 (A), R30.2
- new net: JP7.3 (B), R17.2
- new net: C33.1, JP5.2 (B), L1.1, TP3.1, U11.4 (EN), U11.5 (IN)
- new net: D3.2 (A), L1.2, U11.1 (SW)
- new net BACKLIGHT_POWER: JP6.2 (B), TP4.1
- new net GND: C32.2, C33.2, JP8.2 (C), U11.2 (GND)
Other:
- note added: "LCD backlight power"
- note added: "input: 5v output: 12.8 output voltage is set by changing values of the r17 and r18 ideal values r17: 203k (rare find) r18: 10k"
- company: Grigorii Merkushev (aka brushknight) -> dotstar.tech
- title: Wall panel -> Wall Panel
- moved on the sheet: JP2, TP1, TP2

Commit message: pogo pins wall panel
Parts:
- removed JP7, JP8: 12.8/15V, Jumper:SolderJumper-3_P1.3mm_Bridged12_Pad1.0x1.5mm, symbol Jumper:SolderJumper_3_Bridged12
- removed R17: 200K, Resistor_SMD:R_0402_1005Metric, symbol Device:R_Small
- removed R18: 10K, Resistor_SMD:R_0402_1005Metric, symbol Device:R_Small
- removed TP1, TP2: TestPoint, TestPoint:TestPoint_Pad_D1.5mm, symbol Connector:TestPoint
- removed TP4: boost out, TestPoint:TestPoint_Pad_D1.5mm, symbol Connector:TestPoint
Connections:
- net GND: now also R29.1
- net at C32.1, D3.1 (K), JP6.1 (A): now also R30.2
