File: pcb/wall-panel/power.kicad_sch (KiCad schematic)
At the start: 12 parts, among them U11 MT3608

Commit message: wall panel rev 5
Parts:
- removed C32, C33: 22uF, Capacitor_SMD:C_0805_2012Metric, symbol Device:C_Small
- removed D3: B5817W, Diode_SMD:D_SOD-123, symbol Device:D
- removed JP5, JP6: SolderJumper_2_Bridged, Jumper:SolderJumper-2_P1.3mm_Bridged2Bar_Pad1.0x1.5mm, symbol Jumper:SolderJumper_2_Bridged
- removed L1: 10uH, Inductor_SMD:L_Taiyo-Yuden_NR-40xx, symbol Device:L_Small
- removed R29: 10K, Resistor_SMD:R_0402_1005Metric, symbol Device:R_Small
- removed R30: 240K, Resistor_SMD:R_0402_1005Metric, symbol Device:R_Small
- removed TP3: boost in, TestPoint:TestPoint_Pad_D1.5mm, symbol Connector:TestPoint
- removed TP5: boost fb, TestPoint:TestPoint_Pad_D1.5mm, symbol Connector:TestPoint
- removed U11: MT3608, Package_TO_SOT_SMD:SOT-23-6, symbol Regulator_Switching:MT3608
Other:
- note removed: "LCD backlight power"
- note removed: "input: 5v output: 12.8 output voltage is set by changing values of the r17 and r18 ideal values r17: 203k (rare find) r18: 10k"
