File: pcb/wall-panel/CM4_GPIO.kicad_sch (KiCad schematic)
At the start: 35 parts, among them J10 THD-20-R, J11 pogo_2-1_3, J12 pogo_2-4_6, J13 pogo_2-7_9, J14 pogo_2-10_12, J15 THD-20-R, J16 Micro_SD_Card_Det, J18 THD-20-R, J3 pogo_1-1_3, J7 pogo_1-4_6, J8 pogo_1-7_9, J9 pogo_1-10_12, SW1 power reset, SW2 cpu reset, U10 RT9742GGJ5, U9 74LVC1G07SE-7

Commit message: wall panel rev 5
Connections:
- net GPIO16 is gone; now on net SPI1_CS3: J10.36 (Pin_36), Module1.29 (GPIO16)
- net GPIO17 is gone; now on net SPI1_CS2: J10.11 (Pin_11), Module1.50 (GPIO17)
- net GPIO18 is gone; now on net SPI1_CS1: J10.12 (Pin_12), Module1.49 (GPIO18)
- net GPIO19 is gone; now on net SPI1_MISO: J10.35 (Pin_35), Module1.26 (GPIO19)
- net GPIO20 is gone; now on net SPI1_MOSI: J10.38 (Pin_38), Module1.27 (GPIO20)
- net EEPROM_nWP: now also J11.3 (Pin_3); no longer J3.1 (Pin_1)
- net GPIO27: now also S1.1, S3.1
- net OTG_MODE_SW1: now also J3.2 (Pin_2)
- net USB_OTG_SWITCH: now also J3.1 (Pin_1); no longer J3.2 (Pin_2)
- net SPI1_MISO: now reaches J14.1 (Pin_1)
- net SPI1_MOSI: now reaches J14.2 (Pin_2)
- net SPI1_CS1: now reaches J14.3 (Pin_3)
- net SPI1_SCLK: now reaches J13.3 (Pin_3)
- net SPI1_SCLK: now also J10.40 (Pin_40), Module1.25 (GPIO21)
- net SPI1_CS3: now reaches J9.2 (Pin_2)
- net SPI1_CS2: now reaches J9.3 (Pin_3)
- removed net GPIO21: J10.40 (Pin_40), Module1.25 (GPIO21), S1.1, S3.1
Changed lines of the file:
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@@
 	(title_block
 		(title "Wall Panel")
-		(date "2026-02-25")
-		(rev "v0.3.1")
+		(date "2026-08-24")
+		(rev "5")
 		(company "dotstar.tech")
 		(comment 1 "designed by Grigorii Merkushev (aka brushknight)")
@@
 	(polyline
 		(pts
-			(xy 257.81 130.175) (xy 257.81 168.91)
+			(xy 257.81 130.175) (xy 257.81 239.395)
 		)
 		(stroke
@@
 	(polyline
 		(pts
-			(xy 352.425 130.175) (xy 352.425 168.91)
+			(xy 352.425 130.175) (xy 352.425 239.395)
 		)
 		(stroke
@@
 		)
 	)
+	(label "GPIO27"
+		(at 88.9 241.3 0)
+		(effects
+			(font
+				(size 1.27 1.27)
+			)
+			(justify left bottom)
+		)
+	)
 	(label "GPIO23"
 		(at 124.46 93.98 180)
@@
 		)
 	)
-	(label "GPIO21"
-		(at 88.9 241.3 0)
-		(effects
-			(font
-				(size 1.27 1.27)
-			)
-			(justify left bottom)
-		)
-	)
 	(label "SD_DAT0"
 		(at 125.73 114.3 180)
@@
 		)
 	)
+	(label "GPIO27"
+		(at 88.9 259.08 0)
+		(effects
+			(font
+				(size 1.27 1.27)
+			)
+			(justify left bottom)
+		)
+	)
 	(label "GPIO5"
 		(at 195.58 114.3 180)
@@
 		)
 	)
-	(label "GPIO21"
-		(at 88.9 259.08 0)
-		(effects
-			(font
-				(size 1.27 1.27)
-			)
-			(justify left bottom)
-		)
-	)
 	(label "GPIO27"
 		(at 196.85 93.98 180)
@@
 	)
 	(label "EEPROM_nWP"
-		(at 321.31 179.07 180)
+		(at 288.29 184.15 0)
 		(effects
 			(font
 				(size 1.27 1.27)
 			)
-			(justify right bottom)
+			(justify left bottom)
 		)
 	)
@@
 	(hierarchical_label "USB_OTG_SWITCH"
 		(shape bidirectional)
-		(at 321.31 181.61 180)
+		(at 321.31 179.07 180)
 		(effects
 			(font
@@
 		)
 	)
+	(hierarchical_label "SPI1_MOSI"
+		(shape output)
+		(at 224.79 124.46 0)
+		(effects
+			(font
+				(size 1.27 1.27)
+			)
+			(justify left)
+		)
+	)
 	(hierarchical_label "HD3_P"
 		(shape input)
@@
 		)
 	)
+	(hierarchical_label "SPI1_SCLK"
+		(shape output)
+		(at 224.79 127 0)
+		(effects
+			(font
+				(size 1.27 1.27)
+			)
+			(justify left)
+		)
+	)
+	(hierarchical_label "OTG_MODE_SW1"
+		(shape input)
+		(at 321.31 181.61 180)
+		(effects
+			(font
+				(size 1.27 1.27)
+			)
+			(justify right)
+		)
+	)
 	(hierarchical_label "VBUS"
 		(shape output)
@@
 		)
 	)
+	(hierarchical_label "SPI1_CS2"
+		(shape output)
+		(at 189.23 91.44 180)
+		(effects
+			(font
+				(size 1.27 1.27)
+			)
+			(justify right)
+		)
+	)
+	(hierarchical_label "SPI1_MISO"
+		(shape output)
+		(at 288.29 201.93 0)
+		(effects
+			(font
+				(size 1.27 1.27)
+			)
+			(justify left)
+		)
+	)
 	(hierarchical_label "VBUS"
 		(shape output)
@@
 		)
 	)
+	(hierarchical_label "SPI1_CS1"
+		(shape output)
+		(at 224.79 91.44 0)
+		(effects
+			(font
+				(size 1.27 1.27)
+			)
+			(justify left)
+		)
+	)
 	(hierarchical_label "SDA4"
 		(shape output)
@@
 		)
 	)
+	(hierarchical_label "SPI1_MOSI"
+		(shape output)
+		(at 288.29 204.47 0)
+		(effects
+			(font
+				(size 1.27 1.27)
+			)
+			(justify left)
+		)
+	)
 	(hierarchical_label "SCL1"
 		(shape output)
@@
 		)
 	)
+	(hierarchical_label "SPI1_CS1"
+		(shape output)
+		(at 288.29 207.01 0)
+		(effects
+			(font
+				(size 1.27 1.27)
+			)
+			(justify left)
+		)
+	)
+	(hierarchical_label "SPI1_CS2"
+		(shape output)
+		(at 321.31 207.01 180)
+		(effects
+			(font
+				(size 1.27 1.27)
+			)
+			(justify right)
+		)
+	)
 	(hierarchical_label "UART_RX"
 		(shape output)
@@
 		)
 	)
+	(hierarchical_label "SPI1_SCLK"
+		(shape output)
+		(at 288.29 199.39 0)
+		(effects
+			(font
+				(size 1.27 1.27)
+			)
+			(justify left)
+		)
+	)
 	(hierarchical_label "SCL1"
 		(shape output)
@@
 		)
 	)
+	(hierarchical_label "SPI1_CS3"
+		(shape output)
+		(at 321.31 204.47 180)
+		(effects
+			(font
+				(size 1.27 1.27)
+			)
+			(justify right)
+		)
+	)
 	(hierarchical_label "OTG_MODE_SW1"
 		(shape input)
@@
 		)
 	)
+	(hierarchical_label "SPI1_CS3"
+		(shape output)
+		(at 224.79 121.92 0)
+		(effects
+			(font
+				(size 1.27 1.27)
+			)
+			(justify left)
+		)
+	)
 	(hierarchical_label "ID_SD"
 		(shape output)
@@
 		)
 	)
+	(hierarchical_label "SPI1_MISO"
+		(shape output)
+		(at 189.23 121.92 180)
+		(effects
+			(font
+				(size 1.27 1.27)
+			)
+			(justify right)
+		)
+	)
