File: pcb/wall-panel/CM4_HighSpeed.kicad_sch (KiCad schematic)
At the start: 25 parts, among them J5 SFV30R-4STBE1HLF, J6 690-019-298-412, U12 OC7140, U6 RT9742SNGV, U7 LP5907MFX-2.8, U8 OC7140

Commit message: wall panel rev 5
Parts:
- removed R31, R32: 2.4R, Resistor_SMD:R_0603_1608Metric, symbol Device:R_Small
- removed U12, U8: OC7140, OC7140:ESOP-8, symbol OC7140:OC7140
- added C35: 2.2uF, Capacitor_SMD:C_0603_1608Metric, symbol Device:C_Small
- added C36: 22uF, Capacitor_SMD:C_0805_2012Metric, symbol Device:C_Small
- added C37: 1uF, Capacitor_SMD:C_0603_1608Metric, symbol Device:C_Small
- added D5: SS34, Diode_SMD:D_SMA, symbol Diode:SS34
- added IC2: LM3630ATMX, BGA12C40P3X4_139X191X68, symbol LM3630ATMX:LM3630ATMX
- added JP5, JP6: SolderJumper_2_Bridged, Jumper:SolderJumper-2_P1.3mm_Bridged2Bar_Pad1.0x1.5mm, symbol Jumper:SolderJumper_2_Bridged
- added JP7, JP8: GPIO reference, Jumper:SolderJumper-3_P1.3mm_Bridged12_RoundedPad1.0x1.5mm, symbol Jumper:SolderJumper_3_Bridged12
- added L2: 10uH, CKST0603:IND-SMD_L7.4-W6.6, symbol Device:L_Small
- J5: value SFV30R-4STBE1HLF -> SFV30R-1STBE1HLF; LCSC C3168637 -> C5408677; Manufacturer_Part_Number SFV30R-4STBE1HLF -> SFV30R-1STBE1HLF
Connections:
- net +3.3V: now also IC2.C1 (PWM), JP7.3 (B), JP8.1 (A)
- net +5V: now also JP5.1 (A)
- net BACKLIGHT_POWER: now also JP6.2 (B)
- net GND: now also C35.2, C36.2, C37.2, IC2.B3 (GND), JP7.1 (A), JP8.3 (B)
- net LEDK1: now also IC2.D2 (ILED2)
- net LEDK2: now also IC2.D3 (ILED1)
- net TOUCH_SCL: now also IC2.A2 (SCL)
- net TOUCH_SDA: now also IC2.A1 (SDA)
- new net: C36.1, C37.1, D5.1 (K), IC2.D1 (OVP), JP6.1 (A)
- new net: IC2.B1 (HWEN), JP8.2 (C)
- new net: C35.1, IC2.C3 (IN), JP5.2 (B), L2.1
- new net: D5.2 (A), IC2.A3 (SW), L2.2
- new net: IC2.C2 (SEL), JP7.2 (C)
- no-connect marks 9 -> 3
Other:
- note added: "CM4 High Speed"
- note added: "HDMI"
- note added: "LCD backlight power"
- note added: "MIPI Display"
- note removed: "Jumpers to be fitted if Camera0 or Display0 are used."
- moved on the sheet: C18, C19, C20, C21, C22, C23, C24, C25, C26, C27, C28, C29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
