File: pcb/wall-panel/wall_panel.kicad_pcb (KiCad board)
At the start: 8 copper layers, 75 x 79 mm, 122 parts, among them IC1 TS3USB221RSER, J1 USB_C_Receptacle_USB2.0_14P, J10 THD-20-R, J11 pogo_2-1_3, J12 pogo_2-4_6, J13 pogo_2-7_9, J14 pogo_2-10_12, J16 Micro_SD_Card_Det, J17 USB_C_Receptacle_USB2.0_14P, J2 USB_C_Receptacle_USB2.0_14P, J3 pogo_1-1_3, J4 Conn_01x02_Socket, J5 SFV30R-4STBE1HLF, J7 pogo_1-4_6, J8 pogo_1-7_9, J9 pogo_1-10_12, SW1 power reset, U1 FSUSB42MUX, U10 RT9742GGJ5, U11 MT3608, U12 OC7140, U13 TPD4EUSB30, U2 USB2514B-I/M2, U3 TPD4EUSB30, U4 AP22653W6, U5 DS3231M, U7 LP5907MFX-2.8, U8 OC7140, U9 74LVC1G07SE-7, Y1 ABM8G-24.000MHZ-18-D2Y-T

Commit message: wall panel rev 5
Parts:
- removed C32, C33: 22uF, Capacitor_SMD:C_0805_2012Metric
- removed D3: B5817W, Diode_SMD:D_SOD-123
- removed L1: 10uH, Inductor_SMD:L_Taiyo-Yuden_NR-40xx
- removed R29: 10K, Resistor_SMD:R_0402_1005Metric
- removed R30: 240K, Resistor_SMD:R_0402_1005Metric
- removed R31, R32: 2.4R, Resistor_SMD:R_0603_1608Metric
- removed TP3: boost in, TestPoint:TestPoint_Pad_D1.5mm
- removed TP5: boost fb, TestPoint:TestPoint_Pad_D1.5mm
- removed U11: MT3608, Package_TO_SOT_SMD:SOT-23-6
- removed U12, U8: OC7140, OC7140:ESOP-8
- removed kibuzzard-6A294290: G***, kibuzzard-6A294290
- added C35: 2.2uF, Capacitor_SMD:C_0603_1608Metric, F.Cu at (63.9, 65.2)
- added C36: 22uF, Capacitor_SMD:C_0805_2012Metric, F.Cu at (63.1, 67.7)
- added C37: 1uF, Capacitor_SMD:C_0603_1608Metric, F.Cu at (63.1, 70.9)
- added D5: SS34, Diode_SMD:D_SMA, F.Cu at (67.9, 70.0)
- added IC2: LM3630ATMX, LM3630ATMX:BGA12C40P3X4_139X191X68, F.Cu at (68.8, 66.5)
- added JP7: GPIO reference, Jumper:SolderJumper-3_P1.3mm_Bridged12_RoundedPad1.0x1.5mm, F.Cu at (76.7, 67.6)
- added JP8: GPIO reference, Jumper:SolderJumper-3_P1.3mm_Bridged12_RoundedPad1.0x1.5mm, F.Cu at (74.2, 67.6)
- added L2: 10uH, CKST0603:IND-SMD_L7.4-W6.6, F.Cu at (58.6, 67.7)
- added kibuzzard-6A732F3C: G***, kibuzzard-6A732F3C, B.Cu at (111.5, 129.2)
- moved C31 31.2 mm to (62.9, 95.8), turned to 90 degrees
- moved U10 27.3 mm to (65.9, 95.8), turned to 90 degrees
- moved R22 24.2 mm to (68.4, 95.8), turned to 90 degrees
- moved R20 23.0 mm to (69.4, 95.8), turned to 90 degrees
- moved SW1 14.6 mm to (57.4, 111.6), turned to 0 degrees
- moved kibuzzard-6A266BBE 13.4 mm to (61.6, 112.1)
- moved kibuzzard-6A266BA6 12.7 mm to (68.6, 111.8)
- moved S6 12.5 mm to (68.7, 104.6)
- moved JP5 10.9 mm to (56.1, 75.5), turned to 90 degrees
- moved JP6 6.53 mm to (64.0, 62.6), turned to 0 degrees
- moved R8 1.25 mm to (64.7, 107.1)
- moved R9 1.25 mm to (64.7, 101.3)
- moved U3 1.25 mm to (64.7, 104.3)
Connections:
- J11 pad 3: unconnected-(J11-Pin_3-Pad3) -> /CM4_GPIO ( Ethernet, GPIO, SDCARD)/EEPROM_nWP
- J13 pad 3: unconnected-(J13-Pin_3-Pad3) -> /CM4_GPIO ( Ethernet, GPIO, SDCARD)/GPIO21
- J14 pad 1: unconnected-(J14-Pin_1-Pad1) -> /CM4_GPIO ( Ethernet, GPIO, SDCARD)/GPIO19
- J14 pad 2: unconnected-(J14-Pin_2-Pad2) -> /CM4_GPIO ( Ethernet, GPIO, SDCARD)/GPIO20
- J14 pad 3: unconnected-(J14-Pin_3-Pad3) -> /CM4_GPIO ( Ethernet, GPIO, SDCARD)/GPIO18
- J3 pad 1: /CM4_GPIO ( Ethernet, GPIO, SDCARD)/EEPROM_nWP -> /CM4_GPIO ( Ethernet, GPIO, SDCARD)/USB_OTG_SWITCH
- J3 pad 2: /CM4_GPIO ( Ethernet, GPIO, SDCARD)/USB_OTG_SWITCH -> /CM4_GPIO ( Ethernet, GPIO, SDCARD)/OTG_MODE_SW1
- J9 pad 2: unconnected-(J9-Pin_2-Pad2) -> /CM4_GPIO ( Ethernet, GPIO, SDCARD)/GPIO16
- J9 pad 3: unconnected-(J9-Pin_3-Pad3) -> /CM4_GPIO ( Ethernet, GPIO, SDCARD)/GPIO17
- S1 pad 1: /CM4_GPIO ( Ethernet, GPIO, SDCARD)/GPIO21 -> /CM4_GPIO ( Ethernet, GPIO, SDCARD)/GPIO27
- S3 pad 1: /CM4_GPIO ( Ethernet, GPIO, SDCARD)/GPIO21 -> /CM4_GPIO ( Ethernet, GPIO, SDCARD)/GPIO27
Routing:
- net /CM4_GPIO ( Ethernet, GPIO, SDCARD)/GPIO20: track 52.5 -> 99.4 mm
- net /CM4_HighSpeed/DISPLAY_PWM: track 46.0 -> 0.00 mm, vias 3 -> 1
- net /CM4_GPIO ( Ethernet, GPIO, SDCARD)/GPIO19: track 57.5 -> 101.3 mm, vias 2 -> 4
- net /CM4_GPIO ( Ethernet, GPIO, SDCARD)/GPIO16: track 54.2 -> 97.7 mm, vias 2 -> 4
- net /CM4_GPIO ( Ethernet, GPIO, SDCARD)/GPIO27: track 79.1 -> 121.4 mm, vias 2 -> 4
- net /CM4_HighSpeed/TOUCH_SDA: track 20.4 -> 51.9 mm
- net Net-(J16-DET_A): track 44.0 -> 14.0 mm
- net /CM4_GPIO ( Ethernet, GPIO, SDCARD)/GPIO21: track 129.3 -> 100.8 mm, vias 4 -> 3
- net /CM4_HighSpeed/TOUCH_SCL: track 26.9 -> 52.3 mm
- net Net-(IC2-IN): track 0.25 -> 24.5 mm
- net /CM4_GPIO ( Ethernet, GPIO, SDCARD)/SD_PWR_ON: track 28.0 -> 10.1 mm, vias 2 -> 0
- net Net-(D5-K): track 0.00 -> 16.5 mm, vias 0 -> 10
- net Net-(D5-A): track 0.00 -> 14.8 mm
- net /CM4_GPIO ( Ethernet, GPIO, SDCARD)/GLOBAL_EN: track 34.2 -> 49.0 mm
- net /CM4_GPIO ( Ethernet, GPIO, SDCARD)/SD_PWR: track 34.5 -> 20.0 mm
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- added copper zone on B.Cu, net Net-(D5-K)
- removed copper zone on F.Cu, net Net-(IC2-IN)
